Commit message: Updated turtlebot files to fix teleop.

File: turtlebot3/turtlebot3_description/urdf/turtlebot3_burger.urdf.xacro (robot description, xacro)
@@ -140,7 +140,3 @@
     </inertial>
   </link>
-  <xacro:include filename="$(find turtlebot3_description)/urdf/_d435.urdf.xacro" />
-  <xacro:sensor_d435 parent="base_footprint">
-    <origin xyz="0.0 0.0 0.064" rpy="0.0 0.0 0.0"/>
-  </xacro:sensor_d435>
 </robot>
